Commit message: Add laser link

File: src/rover_description/xacro/rover_platform/rover.gazebo-fortress.xacro (robot description, xacro)
@@ -60,5 +60,5 @@
     <!-- Laser (LiDAR) Joint -->
     <joint name="laser_joint" type="fixed">
-        <origin xyz="0 0 0.2" rpy="0 0 0"/>
+        <origin xyz="0 0 0.4" rpy="0 0 0"/>
         <parent link="chassis_link"/>
         <child link="laser_link"/>
@@ -67,9 +67,9 @@
     <gazebo reference="laser_link">
         <material>Gazebo/Black</material>
-        <sensor name="laser" type="ray">
+        <sensor name="laser" type="gpu_lidar">
             <pose> 0 0 0 0 0 0 </pose>
             <visualize>false</visualize>
             <update_rate>10</update_rate>
-            <ray>
+            <lidar>
                 <scan>
                     <horizontal>
@@ -83,16 +83,11 @@
                     <max>12</max>
                 </range>
-            </ray>
-            <plugin name="laser_controller" filename="libgazebo_ros_ray_sensor.so">
-                <ros>
-                    <argument>~/out:=scan</argument>
-                </ros>
-                <output_type>sensor_msgs/LaserScan</output_type>
-                <frame_name>laser_frame</frame_name>
-            </plugin>
+            </lidar>
+            <topic>scan</topic>
+            <gz_frame_id>laser_link</gz_frame_id>
         </sensor>
     </gazebo>
     <!-- Gazebo Camera Link -->
-    <!-- <link name="camera_link">
+    <link name="camera_link">
         <inertial>
             <origin xyz="0 0 0" rpy="0 0 0"/>
@@ -115,5 +110,5 @@
             </geometry>
         </collision>
-    </link> -->
+    </link>
     <!-- Camera Joint -->
     <joint name="camera_joint" type="fixed">

Commit message: params change

File: src/rover_description/xacro/rover_platform/rover.gazebo-fortress.xacro (robot description, xacro)
@@ -10,7 +10,9 @@
             <right_joint>front_right_wheel_joint</right_joint>
             <right_joint>rear_right_wheel_joint</right_joint>
-            <wheel_radius>0.305</wheel_radius>
+            <wheel_radius>0.3045</wheel_radius>
             <wheel_separation>1.386</wheel_separation>
             <max_linear_acceleration>1.0</max_linear_acceleration>
+            <max_angular_acceleration>1.0</max_angular_acceleration>
+            <max_wheel_torque>10.0</max_wheel_torque>
             <!-- Input -->
             <topic>cmd_vel</topic>

File: src/rover_description/xacro/rover_platform/rover_platform.xacro (robot description, xacro)
@@ -6,5 +6,5 @@
     <xacro:include filename="rover.gazebo-fortress.xacro" />
     <xacro:property name="PI" value="3.1415926535897931" />
-    <xacro:property name="wheel_radius" value="0.3" />
+    <xacro:property name="wheel_radius" value="0.3045" />
     <xacro:property name="wheel_width" value="0.25" />
     <xacro:property name="wheel_mass" value="15" />
@@ -125,5 +125,6 @@
                 <origin xyz="0 0 0" rpy="0 0 ${PI/2}" />
                 <geometry>
-                    <cylinder radius="${wheel_radius}" length="${wheel_width}" />
+                    <!-- <cylinder radius="${wheel_radius}" length="${wheel_width}" /> -->
+                    <mesh filename="package://rover_description/meshes/rover_platform/visuals/wheel.stl" />
                 </geometry>
             </collision>

Commit message: Update

File: src/rover_description/xacro/rover_platform/rover.gazebo-fortress.xacro (robot description, xacro)
@@ -1,4 +1,49 @@
 <?xml version="1.0"?>
 <robot xmlns:xacro="http://www.ros.org/wiki/xacro">
+    <ros2_control name="GazeboSystem" type="system">
+        <hardware>
+            <plugin>ign_ros2_control/IgnitionSystem</plugin>
+        </hardware>
+        <joint name="front_left_wheel_joint">
+            <command_interface name="velocity">
+                <param name="min">-10</param>
+                <param name="max">10</param>
+            </command_interface>
+            <state_interface name="velocity" />
+            <state_interface name="position" />
+        </joint>
+        <joint name="front_right_wheel_joint">
+            <command_interface name="velocity">
+                <param name="min">-10</param>
+                <param name="max">10</param>
+            </command_interface>
+            <state_interface name="velocity" />
+            <state_interface name="position" />
+        </joint>
+        <joint name="rear_left_wheel_joint">
+            <command_interface name="velocity">
+                <param name="min">-10</param>
+                <param name="max">10</param>
+            </command_interface>
+            <state_interface name="velocity" />
+            <state_interface name="position" />
+        </joint>
+        <joint name="rear_right_wheel_joint">
+            <command_interface name="velocity">
+                <param name="min">-10</param>
+                <param name="max">10</param>
+            </command_interface>
+            <state_interface name="velocity" />
+            <state_interface name="position" />
+        </joint>
+    </ros2_control>
+    <gazebo>
+        <plugin filename="ign_ros2_control-system"
+            name="ign_ros2_control::IgnitionROS2ControlPlugin">
+            <robot_param>robot_description</robot_param>
+            <robot_param_node>robot_state_publisher</robot_param_node>
+            <parameters>$(find rover_description)/config/robot_control.yaml</parameters>
+        </plugin>
+    </gazebo>
     <!-- Gazebo Diff Drive -->
     <!-- Simulates a differential drive systems for mobile robot -->
@@ -11,8 +56,7 @@
             <right_joint>rear_right_wheel_joint</right_joint>
             <wheel_radius>0.3045</wheel_radius>
-            <wheel_separation>1.0</wheel_separation>
-            <max_linear_acceleration>0.5</max_linear_acceleration>
-            <max_angular_acceleration>0.2</max_angular_acceleration>
-            <!-- <max_wheel_torque>20.0</max_wheel_torque> -->
+            <wheel_separation>1.25</wheel_separation>
+            <max_linear_acceleration>100.0</max_linear_acceleration>
+            <max_angular_acceleration>100.0</max_angular_acceleration>
             <!-- Input -->
             <topic>cmd_vel</topic>
@@ -21,5 +65,5 @@
             <child_frame_id>base_link</child_frame_id>
             <odom_topic>odom</odom_topic>
-            <odom_publisher_frequency>50</odom_publisher_frequency>
+            <odom_publisher_frequency>30</odom_publisher_frequency>
             <tf_topic>/tf</tf_topic>
         </plugin>

File: src/rover_description/xacro/rover_platform/rover_platform.xacro (robot description, xacro)
@@ -11,5 +11,5 @@
     <xacro:property name="wheel_to_track_ratio" value="0.5962" />
     <xacro:property name="axle_x_offset" value="0.457367" />
-    <xacro:property name="axle_y_offset" value="0.0" />
+    <xacro:property name="axle_y_offset" value="0.5" />
     <xacro:property name="axle_z_offset" value="-0.012977" />
     <xacro:property name="diff_unit_length" value="1.34" />
@@ -23,5 +23,5 @@
     <xacro:property name="chassis_width" value="0.70" />
     <xacro:property name="chassis_height" value="0.30" />
-    <xacro:property name="chassis_mass" value="100" />
+    <xacro:property name="chassis_mass" value="50" />
     <xacro:property name="dummy_inertia" value="1e-09" />
     <xacro:property name="rover_color" value="green" />
@@ -112,5 +112,5 @@
             </inertial>
             <visual>
-                <origin xyz="0 0 0" rpy="0 0 ${PI/2}" />
+                <origin xyz="0 0 0" rpy="0 0 0" />
                 <geometry>
                     <!-- <cylinder radius="${wheel_radius}" length="${wheel_width}" /> -->
@@ -123,5 +123,5 @@
             </visual>
             <collision>
-                <origin xyz="0 0 0" rpy="0 0 ${PI/2}" />
+                <origin xyz="0 0 0" rpy="0 0 0" />
                 <geometry>
                     <!-- <cylinder radius="${wheel_radius}" length="${wheel_width}" /> -->
@@ -138,7 +138,7 @@
     </xacro:macro>
     <!-- Adding Four Wheels -->
-    <xacro:wheel prefix="front" side="left" x="0.5" y="0.5" />
-    <xacro:wheel prefix="front" side="right" x="0.5" y="-0.5" />
-    <xacro:wheel prefix="rear" side="left" x="-0.5" y="0.5" />
-    <xacro:wheel prefix="rear" side="right" x="-0.5" y="-0.5" />
+    <xacro:wheel prefix="front" side="left" x="${axle_x_offset}" y="${axle_y_offset}" />
+    <xacro:wheel prefix="front" side="right" x="${axle_x_offset}" y="${axle_y_offset*-1}" />
+    <xacro:wheel prefix="rear" side="left" x="${axle_x_offset*-1}" y="${axle_y_offset}" />
+    <xacro:wheel prefix="rear" side="right" x="${axle_x_offset*-1}" y="${axle_y_offset*-1}" />
 </robot>

Commit message: modified files

File: src/rover_description/xacro/rover_platform/rover.gazebo-fortress.xacro (robot description, xacro)
@@ -1,73 +1,48 @@
 <?xml version="1.0"?>
 <robot xmlns:xacro="http://www.ros.org/wiki/xacro">
-    <ros2_control name="GazeboSystem" type="system">
-        <hardware>
-            <plugin>ign_ros2_control/IgnitionSystem</plugin>
-        </hardware>
-        <joint name="front_left_wheel_joint">
-            <command_interface name="velocity">
-                <param name="min">-10</param>
-                <param name="max">10</param>
-            </command_interface>
-            <state_interface name="velocity" />
-            <state_interface name="position" />
-        </joint>
-        <joint name="front_right_wheel_joint">
-            <command_interface name="velocity">
-                <param name="min">-10</param>
-                <param name="max">10</param>
-            </command_interface>
-            <state_interface name="velocity" />
-            <state_interface name="position" />
-        </joint>
-        <joint name="rear_left_wheel_joint">
-            <command_interface name="velocity">
-                <param name="min">-10</param>
-                <param name="max">10</param>
-            </command_interface>
-            <state_interface name="velocity" />
-            <state_interface name="position" />
-        </joint>
-        <joint name="rear_right_wheel_joint">
-            <command_interface name="velocity">
-                <param name="min">-10</param>
-                <param name="max">10</param>
-            </command_interface>
-            <state_interface name="velocity" />
-            <state_interface name="position" />
-        </joint>
-    </ros2_control>
-    <gazebo>
-        <plugin filename="ign_ros2_control-system"
-            name="ign_ros2_control::IgnitionROS2ControlPlugin">
-            <robot_param>robot_description</robot_param>
-            <robot_param_node>robot_state_publisher</robot_param_node>
-            <parameters>$(find rover_description)/config/robot_control.yaml</parameters>
-        </plugin>
-    </gazebo>
     <!-- Gazebo Diff Drive -->
     <!-- Simulates a differential drive systems for mobile robot -->
-   <gazebo>
+    <!-- Gazebo Diff Drive -->
+    <gazebo reference="front_left_wheel_joint">
+        <mu1>0.2</mu1>
+        <mu2>0.2</mu2>
+    </gazebo>
+    <gazebo reference="front_right_wheel_joint">
+        <mu1>0.2</mu1>
+        <mu2>0.2</mu2>
+    </gazebo>
+    <gazebo reference="rear_left_wheel_joint">
+        <mu1>0.2</mu1>
+        <mu2>0.2</mu2>
+    </gazebo>
+    <gazebo reference="rear_right_wheel_joint">
+        <mu1>0.2</mu1>
+        <mu2>0.2</mu2>
+    </gazebo>
+       <gazebo>
         <plugin name="gz::sim::systems::DiffDrive" filename="gz-sim-diff-drive-system">
-            <!-- Wheel Information -->
             <left_joint>front_left_wheel_joint</left_joint>
             <left_joint>rear_left_wheel_joint</left_joint>
             <right_joint>front_right_wheel_joint</right_joint>
             <right_joint>rear_right_wheel_joint</right_joint>
+            <wheel_separation>1.7</wheel_separation>
             <wheel_radius>0.3045</wheel_radius>
-            <wheel_separation>1.25</wheel_separation>
-            <max_linear_acceleration>100.0</max_linear_acceleration>
-            <max_angular_acceleration>100.0</max_angular_acceleration>
-            <!-- Input -->
+            <max_wheel_torque>1000</max_wheel_torque>
+            <max_linear_acceleration>1</max_linear_acceleration>
+            <min_linear_acceleration>-1</min_linear_acceleration>
+            <max_angular_acceleration>2</max_angular_acceleration>
+            <min_angular_acceleration>-2</min_angular_acceleration>
+            <max_linear_velocity>0.5</max_linear_velocity>
+            <min_linear_velocity>-0.5</min_linear_velocity>
+            <max_angular_velocity>1</max_angular_velocity>
+            <min_angular_velocity>-1</min_angular_velocity>
             <topic>cmd_vel</topic>
-            <!-- Output -->
             <frame_id>odom</frame_id>
             <child_frame_id>base_link</child_frame_id>
             <odom_topic>odom</odom_topic>
-            <odom_publisher_frequency>30</odom_publisher_frequency>
+            <odom_publisher_frequency>50</odom_publisher_frequency>
             <tf_topic>/tf</tf_topic>
         </plugin>
         <!-- Gazebo Joint States - Used without ROS2 control-->
-        <!-- Publish the state  of the robots joint eg position, velocity to the joint_states topic -->
         <plugin filename="gz-sim-joint-state-publisher-system"
             name="gz::sim::systems::JointStatePublisher">
@@ -77,6 +52,6 @@
             <joint_name>rear_left_wheel_joint</joint_name>
             <joint_name>rear_right_wheel_joint</joint_name>
-            <!-- <joint_name>left_diff_unit_joint</joint_name>
-            <joint_name>right_diff_unit_joint</joint_name> -->
+            <joint_name>left_diff_unit_joint</joint_name>
+            <joint_name>right_diff_unit_joint</joint_name>
         </plugin>
     </gazebo>
@@ -134,61 +109,54 @@
         </sensor>
     </gazebo>
-    <!-- Gazebo Camera Link -->
+    <!-- Camera Link -->
     <link name="camera_link">
-        <inertial>
-            <origin xyz="0 0 0" rpy="0 0 0"/>
-            <mass value="0.1"/>
-            <inertia ixx="0.0001" ixy="0" ixz="0" iyy="0.0001" iyz="0" izz="0.0001"/>
-        </inertial>
         <visual>
-            <origin xyz="0 0 0" rpy="0 0 0"/>
             <geometry>
-                <box size="0.1 0.1 0.1"/>
+                <box size="0.010 0.03 0.03"/>
             </geometry>
-            <material name="red">
-                <color rgba="1 0 0 1"/>
-            </material>
+            <material name="black"/>
         </visual>
-        <collision>
-            <origin xyz="0 0 0" rpy="0 0 0"/>
+        <visual>
+            <origin xyz="0 0 -0.05"/>
             <geometry>
-                <box size="0.1 0.1 0.1"/>
+                <cylinder radius="0.002" length="0.1"/>
             </geometry>
-        </collision>
+            <material name="black"/>
+        </visual>
     </link>
-    <!-- Camera Joint -->
     <joint name="camera_joint" type="fixed">
-        <origin xyz="0.6 0 -0.04" rpy="0 0 0"/>
         <parent link="chassis_link"/>
         <child link="camera_link"/>
+        <origin xyz="0.276 0 1.181" rpy="0 0.18 0"/>
     </joint>
-    <!-- Gazebo Camera Plugin -->
-    <!-- <gazebo reference="laser_frame">
+    <joint name="camera_optical_joint" type="fixed">
+        <parent link="camera_link"/>
+        <child link="camera_link_optical"/>
+        <origin xyz="0 0 0" rpy="${-pi/2} 0 ${-pi/2}"/>
+    </joint>
+    <link name="camera_link_optical"></link>
+    <!-- Gazebo camera plugin -->
+    <gazebo reference="camera_link">
         <material>Gazebo/Black</material>
-        <sensor name="laser" type="ray">
+        <sensor name="camera" type="camera">
             <pose> 0 0 0 0 0 0 </pose>
-            <visualize>false</visualize>
+            <visualize>true</visualize>
             <update_rate>10</update_rate>
-            <ray>
-                <scan>
-                    <horizontal>
-                        <samples>360</samples>
-                        <min_angle>-3.14</min_angle>
-                        <max_angle>3.14</max_angle>
-                    </horizontal>
-                </scan>
-                <range>
-                    <min>0.3</min>
-                    <max>12</max>
-                </range>
-            </ray>
-            <plugin name="laser_controller" filename="libgazebo_ros_ray_sensor.so">
-                <ros>
-                    <argument>~/out:=scan</argument>
-                </ros>
-                <output_type>sensor_msgs/LaserScan</output_type>
-                <frame_name>laser_frame</frame_name>
-            </plugin>
+            <camera>
+                <camera_info_topic>camera/camera_info</camera_info_topic>
+                <horizontal_fov>1.089</horizontal_fov>
+                <image>
+                    <format>R8G8B8</format>
+                    <width>640</width>
+                    <height>480</height>
+                </image>
+                <clip>
+                    <near>0.05</near>
+                    <far>8.0</far>
+                </clip>
+            </camera>
+            <topic>camera/image_raw</topic>
+            <gz_frame_id>camera_link_optical</gz_frame_id>
         </sensor>
-    </gazebo>  -->
+    </gazebo>
 </robot>

Commit message: imu link and plugin added

File: src/rover_description/xacro/rover_platform/rover.gazebo-fortress.xacro (robot description, xacro)
@@ -160,3 +160,18 @@
         </sensor>
     </gazebo>
+    <!-- IMU Link-->
+    <link name="imu_link"></link>
+    <joint name="imu_link_joint" type="fixed">
+        <origin xyz="$(optenv ROVER_IMU_XYZ 0 0 0)" rpy="$(optenv ROVER_IMU_RPY 0 0 0)" />
+        <parent link="chassis_link" />
+        <child link="imu_link" />
+    </joint>
+    <gazebo reference="imu_link">
+        <sensor name="imu_sensor" type="imu">
+            <always_on>1</always_on>
+            <update_rate>1</update_rate>
+            <visualize>true</visualize>
+            <topic>imu</topic>
+        </sensor>
+    </gazebo>
 </robot>

File: src/rover_description/xacro/rover_platform/rover_platform.xacro (robot description, xacro)
@@ -97,10 +97,4 @@
         </collision>
     </link>
-    <link name="imu_link"></link>
-    <joint name="imu_link_joint" type="fixed">
-        <origin xyz="$(optenv ROVER_IMU_XYZ 0 0 0)" rpy="$(optenv ROVER_IMU_RPY 0 0 0)" />
-        <parent link="chassis_link" />
-        <child link="imu_link" />
-    </joint>
     <!-- Wheel Macro -->
     <xacro:macro name="wheel" params="prefix side x y">
